Commit message: made floor bigger

File: assets/short_floor.urdf (robot description, URDF)
Before this commit: robot flat_terrain, 1 links, 0 joints
Links:
- link base_link: geometry collision box size=4 4 0.1; visual box size=4 4 0.1

Commit message: added floor back to make pick/place exercise work

File: assets/short_floor.urdf (robot description, URDF)
Before this commit: robot flat_terrain, 1 links, 0 joints
Links:
- link base_link: geometry collision box size=2 2 0.1; visual box size=2 2 0.1
